Commit message: added a touch sensor

File: urdf/r2d2.urdf.xacro (robot description, xacro)
@@ -9,16 +9,17 @@
   <xacro:property name="pi" value="3.1415" />
   <material name="blue">
-    <color rgba="0 0 0.8 1"/>
+    <color rgba="0 0 0.8 1" />
   </material>
   <material name="black">
-    <color rgba="0 0 0 1"/>
+    <color rgba="0 0 0 1" />
   </material>
   <material name="white">
-    <color rgba="1 1 1 1"/>
+    <color rgba="1 1 1 1" />
   </material>
   <xacro:macro name="default_inertial" params="mass">
     <inertial>
       <mass value="${mass}" />
-      <inertia ixx="1.0" ixy="0.0" ixz="0.0" iyy="1.0" iyz="0.0" izz="1.0" />
+      <inertia ixx="1.0" ixy="0.0" ixz="0.0" iyy="1.0" iyz="0.0"
+      izz="1.0" />
     </inertial>
   </xacro:macro>
@@ -26,14 +27,14 @@
     <visual>
       <geometry>
-        <cylinder radius="${width}" length="${bodylen}"/>
-      </geometry>
-      <material name="blue"/>
+        <cylinder radius="${width}" length="${bodylen}" />
+      </geometry>
+      <material name="blue" />
     </visual>
     <collision>
       <geometry>
-        <cylinder radius="${width}" length="${bodylen}"/>
+        <cylinder radius="${width}" length="${bodylen}" />
       </geometry>
     </collision>
-    <xacro:default_inertial mass="10"/>
+    <xacro:default_inertial mass="10" />
   </link>
   <xacro:macro name="wheel" params="prefix suffix reflect">
@@ -42,27 +43,29 @@
         <origin xyz="0 0 0" rpy="${pi/2} 0 0" />
         <geometry>
-          <cylinder radius="${wheeldiam/2}" length="0.1"/>
-        </geometry>
-        <material name="black"/>
+          <cylinder radius="${wheeldiam/2}" length="0.1" />
+        </geometry>
+        <material name="black" />
       </visual>
       <collision>
         <origin xyz="0 0 0" rpy="${pi/2} 0 0" />
         <geometry>
-          <cylinder radius="${wheeldiam/2}" length="0.1"/>
-        </geometry>
-      </collision>
-      <xacro:default_inertial mass="1"/>
-    </link>
-    <joint name="${prefix}_${suffix}_wheel_joint" type="continuous">
+          <cylinder radius="${wheeldiam/2}" length="0.1" />
+        </geometry>
+      </collision>
+      <xacro:default_inertial mass="5" />
+    </link>
+    <joint name="${prefix}_${suffix}_wheel_joint"
+    type="continuous">
       <axis xyz="0 1 0" rpy="0 0 0" />
-      <parent link="${prefix}_base"/>
-      <child link="${prefix}_${suffix}_wheel"/>
-      <origin xyz="${baselen*reflect/3} 0 -${wheeldiam/2+.05}" rpy="0 0 0"/>
+      <parent link="${prefix}_base" />
+      <child link="${prefix}_${suffix}_wheel" />
+      <origin xyz="${baselen*reflect/3} 0 -${wheeldiam/2+.05}"
+      rpy="0 0 0" />
     </joint>
     <!-- This block provides the simulator (Gazebo) with information on a few additional
     physical properties. See http://gazebosim.org/tutorials/?tut=ros_urdf for more-->
     <gazebo reference="${prefix}_${suffix}_wheel">
-      <mu1 value="200.0"/>
-      <mu2 value="100.0"/>
+      <mu1 value="200.0" />
+      <mu2 value="100.0" />
       <kp value="10000000.0" />
       <kd value="1.0" />
@@ -77,5 +80,6 @@
       </actuator>
       <joint name="${prefix}_${suffix}_wheel_joint">
-        <hardwareInterface>VelocityJointInterface</hardwareInterface>
+        <hardwareInterface>
+        VelocityJointInterface</hardwareInterface>
       </joint>
     </transmission>
@@ -85,20 +89,20 @@
       <visual>
         <geometry>
-          <box size="${leglen} 0.1 0.2"/>
-        </geometry>
-        <origin xyz="0 0 -${leglen/2}" rpy="0 ${pi/2} 0"/>
-        <material name="white"/>
-      </visual>
-      <collision>
-        <geometry>
-          <box size="${leglen} 0.1 0.2"/>
-        </geometry>
-        <origin xyz="0 0 -${leglen/2}" rpy="0 ${pi/2} 0"/>
-      </collision>
-      <xacro:default_inertial mass="10"/>
+          <box size="${leglen} 0.1 0.2" />
+        </geometry>
+        <origin xyz="0 0 -${leglen/2}" rpy="0 ${pi/2} 0" />
+        <material name="white" />
+      </visual>
+      <collision>
+        <geometry>
+          <box size="${leglen} 0.1 0.2" />
+        </geometry>
+        <origin xyz="0 0 -${leglen/2}" rpy="0 ${pi/2} 0" />
+      </collision>
+      <xacro:default_inertial mass="20" />
     </link>
     <joint name="base_to_${prefix}_leg" type="fixed">
-      <parent link="base_link"/>
-      <child link="${prefix}_leg"/>
+      <parent link="base_link" />
+      <child link="${prefix}_leg" />
       <origin xyz="0 ${reflect*(width+.02)} 0.25" />
     </joint>
@@ -106,109 +110,139 @@
       <visual>
         <geometry>
-          <box size="${baselen} 0.1 0.1"/>
-        </geometry>
-        <material name="white"/>
-      </visual>
-      <collision>
-        <geometry>
-          <box size="${baselen} 0.1 0.1"/>
-        </geometry>
-      </collision>
-      <xacro:default_inertial mass="10"/>
+          <box size="${baselen} 0.1 0.1" />
+        </geometry>
+        <material name="white" />
+      </visual>
+      <collision>
+        <geometry>
+          <box size="${baselen} 0.1 0.1" />
+        </geometry>
+      </collision>
+      <xacro:default_inertial mass="30" />
     </link>
     <joint name="${prefix}_base_joint" type="fixed">
-      <parent link="${prefix}_leg"/>
-      <child link="${prefix}_base"/>
+      <parent link="${prefix}_leg" />
+      <child link="${prefix}_base" />
       <origin xyz="0 0 ${-leglen}" />
     </joint>
-    <xacro:wheel prefix="${prefix}" suffix="front" reflect="1"/>
-    <xacro:wheel prefix="${prefix}" suffix="back" reflect="-1"/>
+    <xacro:wheel prefix="${prefix}" suffix="front" reflect="1" />
+    <xacro:wheel prefix="${prefix}" suffix="back" reflect="-1" />
   </xacro:macro>
   <xacro:leg prefix="right" reflect="-1" />
   <xacro:leg prefix="left" reflect="1" />
   <joint name="gripper_extension" type="prismatic">
-    <parent link="base_link"/>
-    <child link="gripper_pole"/>
-    <limit effort="1000.0" lower="-${width*2-.02}" upper="0" velocity="0.5"/>
-    <origin rpy="0 0 0" xyz="${width-.01} 0 0.2"/>
-    <limit effort="30" velocity="0.2"/>
-    <dynamics damping="0.0" friction="0.0"/>
+    <parent link="base_link" />
+    <child link="gripper_pole" />
+    <limit effort="1000.0" lower="-${width*2-.02}" upper="0"
+    velocity="0.5" />
+    <origin rpy="0 0 0" xyz="${width-.01} 0 0.2" />
+    <limit effort="30" velocity="0.2" />
+    <dynamics damping="0.0" friction="0.0" />
   </joint>
   <link name="gripper_pole">
     <visual>
       <geometry>
-        <cylinder length="${polelen}" radius="0.01"/>
-      </geometry>
-      <origin xyz="${polelen/2} 0 0" rpy="0 ${pi/2} 0 "/>
+        <cylinder length="${polelen}" radius="0.01" />
+      </geometry>
+      <origin xyz="${polelen/2} 0 0" rpy="0 ${pi/2} 0" />
     </visual>
     <collision>
       <geometry>
-        <cylinder length="${polelen}" radius="0.01"/>
-      </geometry>
-      <origin xyz="${polelen/2} 0 0" rpy="0 ${pi/2} 0 "/>
+        <cylinder length="${polelen}" radius="0.01" />
+      </geometry>
+      <origin xyz="${polelen/2} 0 0" rpy="0 ${pi/2} 0" />
     </collision>
-    <xacro:default_inertial mass="0.05"/>
+    <xacro:default_inertial mass="0.033" />
   </link>
   <!--<transmission name="gripper_extension_trans">-->
-    <!--<type>transmission_interface/SimpleTransmission</type>-->
-    <!--<actuator name="gripper_extension_motor">-->
-      <!--<mechanicalReduction>1</mechanicalReduction>-->
-    <!--</actuator>-->
-    <!--<joint name="gripper_extension">-->
-      <!--<hardwareInterface>PositionJointInterface</hardwareInterface>-->
-    <!--</joint>-->
+  <!--<type>transmission_interface/SimpleTransmission</type>-->
+  <!--<actuator name="gripper_extension_motor">-->
+  <!--<mechanicalReduction>1</mechanicalReduction>-->
+  <!--</actuator>-->
+  <!--<joint name="gripper_extension">-->
+  <!--<hardwareInterface>PositionJointInterface</hardwareInterface>-->
+  <!--</joint>-->
   <!--</transmission>-->
   <xacro:macro name="gripper" params="prefix reflect">
     <joint name="${prefix}_gripper_joint" type="revolute">
-      <axis xyz="0 0 ${reflect}"/>
-      <limit effort="1000.0" lower="0.0" upper="0.548" velocity="0.5"/>
-      <origin rpy="0 0 0" xyz="${polelen} ${reflect*0.01} 0"/>
-      <parent link="gripper_pole"/>
-      <child link="${prefix}_gripper"/>
-      <limit effort="30" velocity="1.0"/>
-      <dynamics damping="0.0" friction="0.0"/>
+      <axis xyz="0 0 ${reflect}" />
+      <limit effort="1000.0" lower="0.0" upper="0.548"
+      velocity="0.5" />
+      <origin rpy="0 0 0" xyz="${polelen} ${reflect*0.01} 0" />
+      <parent link="gripper_pole" />
+      <child link="${prefix}_gripper" />
+      <limit effort="30" velocity="1.0" />
+      <dynamics damping="0.0" friction="0.0" />
     </joint>
     <link name="${prefix}_gripper">
       <visual>
-        <origin rpy="${(reflect-1)/2*pi} 0 0" xyz="0 0 0"/>
-        <geometry>
-          <mesh filename="package://urdf_tutorial/meshes/l_finger.dae"/>
-        </geometry>
-      </visual>
-      <collision>
-        <geometry>
-          <mesh filename="package://urdf_tutorial/meshes/l_finger.dae"/>
-        </geometry>
-        <origin rpy="${(reflect-1)/2*pi} 0 0" xyz="0 0 0"/>
-      </collision>
-      <xacro:default_inertial mass="0.05"/>
+        <origin rpy="${(reflect-1)/2*pi} 0 0" xyz="0 0 0" />
+        <geometry>
+          <mesh filename="package://urdf_tutorial/meshes/l_finger.dae" />
+        </geometry>
+      </visual>
+      <!--<sensor name="${prefix}_finger_sensor" type="contact">-->
+      <!--<contact>-->
+      <!--<collision>${prefix}_finger_colision</collision>-->
+      <!--</contact>-->
+      <!--</sensor>-->
+      <collision>
+        <geometry>
+          <mesh filename="package://urdf_tutorial/meshes/l_finger.dae" />
+        </geometry>
+        <origin rpy="${(reflect-1)/2*pi} 0 0" xyz="0 0 0" />
+        <surface>
+          <friction>
+            <ode>
+              <mu>2.0</mu>
+              <mu2>2.0</mu2>
+            </ode>
+          </friction>
+        </surface>
+      </collision>
+      <xacro:default_inertial mass="0.05" />
     </link>
     <!--<transmission name="${prefix}_gripper_trans">-->
-      <!--<type>transmission_interface/SimpleTransmission</type>-->
-      <!--<actuator name="${prefix}_gripper_motor">-->
-        <!--<mechanicalReduction>1</mechanicalReduction>-->
-      <!--</actuator>-->
-      <!--<joint name="${prefix}_gripper_joint">-->
-        <!--<hardwareInterface>PositionJointInterface</hardwareInterface>-->
-      <!--</joint>-->
+    <!--<type>transmission_interface/SimpleTransmission</type>-->
+    <!--<actuator name="${prefix}_gripper_motor">-->
+    <!--<mechanicalReduction>1</mechanicalReduction>-->
+    <!--</actuator>-->
+    <!--<joint name="${prefix}_gripper_joint">-->
+    <!--<hardwareInterface>PositionJointInterface</hardwareInterface>-->
+    <!--</joint>-->
     <!--</transmission>-->
     <joint name="${prefix}_tip_joint" type="fixed">
-      <parent link="${prefix}_gripper"/>
-      <child link="${prefix}_tip"/>
+      <parent link="${prefix}_gripper" />
+      <child link="${prefix}_tip" />
     </joint>
     <link name="${prefix}_tip">
       <visual>
-        <origin rpy="${(reflect-1)/2*pi} 0 0" xyz="0.09137 0.00495 0"/>
-        <geometry>
-          <mesh filename="package://urdf_tutorial/meshes/l_finger_tip.dae"/>
-        </geometry>
-      </visual>
-      <collision>
-        <geometry>
-          <mesh filename="package://urdf_tutorial/meshes/l_finger_tip.dae"/>
-        </geometry>
-        <origin rpy="${(reflect-1)/2*pi} 0 0" xyz="0.09137 0.00495 0"/>
-      </collision>
-      <xacro:default_inertial mass="0.05"/>
+        <origin rpy="${(reflect-1)/2*pi} 0 0"
+        xyz="0.09137 0.00495 0" />
+        <geometry>
+          <mesh filename="package://urdf_tutorial/meshes/l_finger_tip.dae" />
+        </geometry>
+      </visual>
+      <!--<sensor name="${prefix}_finger_tip_sensor" type="contact">-->
+      <!--<contact>-->
+      <!--<collision>${prefix}_finger_tip_colision</collision>-->
+      <!--</contact>-->
+      <!--</sensor>-->
+      <collision>
+        <geometry>
+          <mesh filename="package://urdf_tutorial/meshes/l_finger_tip.dae" />
+        </geometry>
+        <origin rpy="${(reflect-1)/2*pi} 0 0"
+        xyz="0.09137 0.00495 0" />
+        <surface>
+          <friction>
+            <ode>
+              <mu>2.0</mu>
+              <mu2>2.0</mu2>
+            </ode>
+          </friction>
+        </surface>
+      </collision>
+      <xacro:default_inertial mass="0.05" />
     </link>
   </xacro:macro>
@@ -218,22 +252,22 @@
     <visual>
       <geometry>
-        <sphere radius="${width}"/>
-      </geometry>
-      <material name="white"/>
+        <sphere radius="${width}" />
+      </geometry>
+      <material name="white" />
     </visual>
     <collision>
       <geometry>
-        <sphere radius="${width}"/>
+        <sphere radius="${width}" />
       </geometry>
     </collision>
-    <xacro:default_inertial mass="2"/>
+    <xacro:default_inertial mass="2" />
   </link>
   <joint name="head_swivel" type="continuous">
-    <parent link="base_link"/>
-    <child link="head"/>
-    <axis xyz="0 0 1"/>
-    <origin xyz="0 0 ${bodylen/2}"/>
-    <limit effort="30" velocity="1.0"/>
-    <dynamics damping="0.0" friction="0.0"/>
+    <parent link="base_link" />
+    <child link="head" />
+    <axis xyz="0 0 1" />
+    <origin xyz="0 0 ${bodylen/2}" />
+    <limit effort="30" velocity="1.0" />
+    <dynamics damping="0.0" friction="0.0" />
   </joint>
   <!-- This block connects the head_swivel joint to an actuator (motor), which informs both
@@ -251,30 +285,34 @@
     <visual>
       <geometry>
-        <box size="0.08 0.08 0.08"/>
-      </geometry>
-      <material name="blue"/>
-      <origin xyz="-0.04 0 0"/>
+        <box size="0.08 0.08 0.08" />
+      </geometry>
+      <material name="blue" />
+      <origin xyz="-0.04 0 0" />
     </visual>
     <collision>
       <geometry>
-        <box size="0.08 0.08 0.08"/>
+        <box size="0.08 0.08 0.08" />
       </geometry>
     </collision>
-    <xacro:default_inertial mass="1"/>
+    <xacro:default_inertial mass="1" />
   </link>
   <joint name="tobox" type="fixed">
-    <parent link="head"/>
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
Commit message: add touch sensor. partially implement force detection

File: urdf/r2d2.urdf.xacro (robot description, xacro)
@@ -182,9 +182,4 @@
         </geometry>
       </visual>
-      <!--<sensor name="${prefix}_finger_sensor" type="contact">-->
-      <!--<contact>-->
-      <!--<collision>${prefix}_finger_colision</collision>-->
-      <!--</contact>-->
-      <!--</sensor>-->
       <collision>
         <geometry>
@@ -201,4 +196,14 @@
         </surface>
       </collision>
+      <!--<gazebo reference="left_gripper">-->
+      <!--<sensor name="gripper_contact_sensor" type="contact">-->
+      <!--<pose>0.0 0.0 0.0 0.0 0 0</pose>-->
+      <!--<visualize>false</visualize>-->
+      <!--<update_rate>5</update_rate>-->
+      <!--<contact>-->
+      <!--<collision name="${prefix}_finger" />-->
+      <!--</contact>-->
+      <!--</sensor>-->
+      <!--</gazebo>-->
       <xacro:default_inertial mass="0.05" />
     </link>
@@ -226,8 +231,9 @@
       <!--<sensor name="${prefix}_finger_tip_sensor" type="contact">-->
       <!--<contact>-->
-      <!--<collision>${prefix}_finger_tip_colision</collision>-->
+      <!--<collision>finger_tip_colision</collision>-->
       <!--</contact>-->
+      <!--<update_rate>5</update_rate>-->
       <!--</sensor>-->
-      <collision>
+      <collision name="finger_tip_colision">
         <geometry>
           <mesh filename="package://urdf_tutorial/meshes/l_finger_tip.dae" />
@@ -310,7 +316,4 @@
       <robotNamespace>/gripper/</robotNamespace>
     </plugin>
-    <!--<plugin name="r2_touch" filename="libr2_touch.so">-->
-    <!--<robotNamespace>/touch/</robotNamespace>-->
-    <!--</plugin>-->
     <plugin name="gazebo_ros_control"
     filename="libgazebo_ros_control.so">
@@ -318,3 +321,31 @@
     </plugin>
   </gazebo>
+  <gazebo reference="left_gripper">
+    <sensor name="left_gripper_contact_sensor" type="contact">
+      <always_on>true</always_on>
+      <visualize>false</visualize>
+      <update_rate>5</update_rate>
+      <contact>
+        <collision>collision</collision>
+      </contact>
+      <plugin name="r2_touch" filename="libr2_touch.so">
+        <robotNamespace>
+        /left_gripper_contact_sensor/</robotNamespace>
+      </plugin>
+    </sensor>
+  </gazebo>
+  <gazebo reference="right_gripper">
+    <sensor name="right_gripper_contact_sensor" type="contact">
+      <always_on>true</always_on>
+      <visualize>false</visualize>
+      <update_rate>5</update_rate>
+      <contact>
+        <collision>collision</collision>
+      </contact>
+      <plugin name="r2_touch" filename="libr2_touch.so">
+        <robotNamespace>
+        /right_gripper_contact_sensor/</robotNamespace>
+      </plugin>
+    </sensor>
+  </gazebo>
 </robot>
